Commit message: Update onrobot_rg2.xacro

File: onrobot_rg_description/urdf/onrobot_rg2.xacro (robot description, xacro)
@@ -24,10 +24,10 @@
       </collision>
     </link>
-    <link name="world"/>
+    <!-- <link name="world"/>
     <joint name="joint0" type="fixed">
         <parent link="world"/>
         <child link="${prefix}onrobot_rg2_base_link"/>
         <origin xyz= "0. 0. 0." rpy="0. 0. 0." />
-    </joint>
+    </joint> -->
     <gazebo reference="${prefix}onrobot_rg2_base_link">
       <mu1>1.0</mu1>
